File: ali/v2/pressuretransducers/pressuretransducers.kicad_sch (KiCad schematic)
At the start: 4 parts

Commit message: Big changes (Tim and Daniel review part 1)
Parts:
- H1, H2, H3, H4: footprint MountingHole:MountingHole_3.2mm_M3 -> APRL_Misc:MountingHole_3.2mm_M3
Changed lines of the file:
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@@
 			)
 		)
-		(property "Footprint" "MountingHole:MountingHole_3.2mm_M3"
+		(property "Footprint" "APRL_Misc:MountingHole_3.2mm_M3"
 			(at 22.86 180.34 0)
 			(hide yes)
@@
 			)
 		)
-		(property "Footprint" "MountingHole:MountingHole_3.2mm_M3"
+		(property "Footprint" "APRL_Misc:MountingHole_3.2mm_M3"
 			(at 22.86 190.5 0)
 			(hide yes)
@@
 			)
 		)
-		(property "Footprint" "MountingHole:MountingHole_3.2mm_M3"
+		(property "Footprint" "APRL_Misc:MountingHole_3.2mm_M3"
 			(at 22.86 195.58 0)
 			(hide yes)
@@
 			)
 		)
-		(property "Footprint" "MountingHole:MountingHole_3.2mm_M3"
+		(property "Footprint" "APRL_Misc:MountingHole_3.2mm_M3"
 			(at 22.86 185.42 0)
 			(hide yes)
