File: ali/v2/pressuretransducers/pressuretransducers.kicad_pcb (KiCad board)
At the start: 4 copper layers, 85 x 76 mm, 183 parts, among them J1 Conn_02x01, J10 Conn_01x02, J11 Conn_01x02, J12 Conn_01x02, J13 Conn_01x02, J14 Conn_01x02, J15 Conn_01x02, J16 Conn_01x02, J17 Conn_01x02, J18 Conn_01x02, J19 Conn_01x02, J2 Conn_01x05, J20 Conn_01x02, J21 Conn_01x02, J22 Conn_01x02, J23 Conn_01x02, J24 Conn_01x02, J25 Conn_01x02, J3 USB_C_Receptacle_USB2.0_16P, J4 Conn_02x09_Counter_Clockwise, J5 Conn_01x15, J6 Screw_Terminal_01x02, J7 Screw_Terminal_01x02, J8 Vertical Ethernet, J9 Conn_01x03, SW1 SKRPANE010, U1 STM32H563RIV6, U2 AP2112K-3.3, U3 LAN8742AI, U4 TJA1462ATK, U5 ADS131M08IRSN, U6 ADS131M08IRSN, Y1 25 MHz, Y2 25 MHz, Y3 8.192 MHz, Y4 8.192 MHz

Commit message: Small cleanups
Parts:
- C29, C30, C35, C37, C38, C41, C43, C44, C45, C46, C51, C53, C54, C57, C59, C60: value 1nF -> 10nF
Routing:
- net GND: vias 439 -> 457
Other:
- board text added: "1/2"
- board text added: "11/12"
- board text added: "13/14"
- board text added: "15/16"
- board text added: "3/4"
- board text added: "5/6"
- board text added: "7/8"
- board text added: "9/10"

Commit message: Big changes (Tim and Daniel review part 1)
Parts:
- added F12: 100mA, APRL_Passive:Fuse_1206_3216Metric, B.Cu at (105.5, 91.5)
- added F13: 100mA, APRL_Passive:Fuse_1206_3216Metric, B.Cu at (105.7, 120.1)
- added F14: 100mA, APRL_Passive:Fuse_1206_3216Metric, B.Cu at (99.1, 91.5)
- added F15: 100mA, APRL_Passive:Fuse_1206_3216Metric, B.Cu at (99.1, 120.1)
- added F16: 100mA, APRL_Passive:Fuse_1206_3216Metric, B.Cu at (105.5, 98.7)
- added F17: 100mA, APRL_Passive:Fuse_1206_3216Metric, B.Cu at (105.7, 127.7)
- added F18: 100mA, APRL_Passive:Fuse_1206_3216Metric, B.Cu at (99.1, 98.7)
- added F19: 100mA, APRL_Passive:Fuse_1206_3216Metric, B.Cu at (99.1, 127.7)
- C11: moved to B.Cu
- H1, H2, H3, H4: footprint MountingHole:MountingHole_3.2mm_M3 -> APRL_Misc:MountingHole_3.2mm_M3
- J6, J7: footprint Connector_Phoenix_MSTB:PhoenixContact_MSTBV_2,5_2-GF-5,08_1x02_P5.08mm_Vertical_ThreadedFlange_MountHole -> APRL_Connector:PhoenixContact_MSTBV_2,5_2-GF-5,08_1x02_P5.08mm_Vertical_ThreadedFlange_MountHole
- moved F10 33.1 mm to (99.1, 84.1), turned to 180 degrees
- moved F6 18.3 mm to (99.1, 105.7), turned to 180 degrees
- moved F11 11.9 mm to (99.1, 113.1), turned to 180 degrees
- moved F7 11.3 mm to (105.5, 84.1), turned to 180 degrees
- moved F5 5.86 mm to (99.1, 77.3), turned to 180 degrees
- moved F4 4.17 mm to (105.7, 77.3), turned to 180 degrees
- moved F9 3.94 mm to (105.7, 113.1), turned to 180 degrees
- moved F8 3.78 mm to (105.7, 105.7), turned to 180 degrees
- moved C11 2.06 mm to (144.2, 93.2), turned to 0 degrees
- moved C36 1.54 mm to (126.6, 90.4), turned to 0 degrees
- moved C52 0.50 mm to (126.4, 120.3)
Connections:
- F10 pad 1: Net-(J22-Pin_2) -> Net-(J13-Pin_2)
- F11 pad 1: Net-(J24-Pin_2) -> Net-(J21-Pin_2)
- F5 pad 1: Net-(J12-Pin_2) -> Net-(J11-Pin_2)
- F6 pad 1: Net-(J14-Pin_2) -> Net-(J19-Pin_2)
- F7 pad 1: Net-(J16-Pin_2) -> Net-(J12-Pin_2)
- J11 pad 2: Net-(J10-Pin_2) -> Net-(J11-Pin_2)
- J13 pad 2: Net-(J12-Pin_2) -> Net-(J13-Pin_2)
- J15 pad 2: Net-(J14-Pin_2) -> Net-(J15-Pin_2)
- J17 pad 2: Net-(J16-Pin_2) -> Net-(J17-Pin_2)
- J19 pad 2: Net-(J18-Pin_2) -> Net-(J19-Pin_2)
- J21 pad 2: Net-(J20-Pin_2) -> Net-(J21-Pin_2)
- J23 pad 2: Net-(J22-Pin_2) -> Net-(J23-Pin_2)
- J25 pad 2: Net-(J24-Pin_2) -> Net-(J25-Pin_2)
Routing:
- net GND: track 7.77 -> 18.1 mm, vias 457 -> 528
- net +5V: track 25.3 -> 20.1 mm, vias 8 -> 11
- net Net-(J11-Pin_2): track 0.00 -> 2.85 mm
- net Net-(J25-Pin_2): track 0.00 -> 2.76 mm
- net Net-(J10-Pin_2): track 0.00 -> 2.71 mm
- net Net-(J15-Pin_2): track 0.00 -> 2.62 mm
- net Net-(J24-Pin_2): track 0.00 -> 2.61 mm
- net Net-(J17-Pin_2): track 0.00 -> 2.60 mm
- net Net-(J21-Pin_2): track 0.00 -> 2.60 mm
- net Net-(J20-Pin_2): track 0.00 -> 2.45 mm
- net Net-(J13-Pin_2): track 0.00 -> 2.44 mm
- net Net-(J19-Pin_2): track 0.00 -> 2.41 mm
- net Net-(J14-Pin_2): track 0.00 -> 2.39 mm
- net Net-(J16-Pin_2): track 0.00 -> 2.37 mm
- net Net-(J23-Pin_2): track 0.00 -> 2.37 mm
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- removed copper zone on B.Cu, net Net-(J10-Pin_2)
- removed copper zone on B.Cu, net Net-(J12-Pin_2)
- removed copper zone on B.Cu, net Net-(J14-Pin_2)
- removed copper zone on B.Cu, net Net-(J16-Pin_2)
- removed copper zone on B.Cu, net Net-(J18-Pin_2)
- removed copper zone on B.Cu, net Net-(J20-Pin_2)
- removed copper zone on B.Cu, net Net-(J22-Pin_2)
- removed copper zone on B.Cu, net Net-(J24-Pin_2)
