File: ali/v2/pressuretransducers/analog.kicad_sch (KiCad schematic)
At the start: 54 parts, among them J10 Conn_01x02, J11 Conn_01x02, J12 Conn_01x02, J13 Conn_01x02, J14 Conn_01x02, J15 Conn_01x02, J16 Conn_01x02, J17 Conn_01x02, U5 ADS131M08IRSN, Y3 8.192 MHz

Commit message: Small cleanups
Parts:
- C29, C30, C35, C37, C38, C41, C43, C44: value 1nF -> 10nF; MPN GRM1885C1H102FA01 -> GRM1885C1H103JA01
Changed lines of the file:
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@@
 			)
 		)
-		(property "Value" "1nF"
+		(property "Value" "10nF"
 			(at 69.85 59.6835 0)
 			(show_name no)
@@
 			)
 		)
-		(property "MPN" "GRM1885C1H102FA01"
+		(property "MPN" "GRM1885C1H103JA01"
 			(at 67.31 58.42 0)
 			(hide yes)
@@
 			)
 		)
-		(property "Value" "1nF"
+		(property "Value" "10nF"
 			(at 69.85 161.2835 0)
 			(show_name no)
@@
 			)
 		)
-		(property "MPN" "GRM1885C1H102FA01"
+		(property "MPN" "GRM1885C1H103JA01"
 			(at 67.31 160.02 0)
 			(hide yes)
@@
 			)
 		)
-		(property "Value" "1nF"
+		(property "Value" "10nF"
 			(at 69.85 179.0635 0)
 			(show_name no)
@@
 			)
 		)
-		(property "MPN" "GRM1885C1H102FA01"
+		(property "MPN" "GRM1885C1H103JA01"
 			(at 67.31 177.8 0)
 			(hide yes)
@@
 			)
 		)
-		(property "Value" "1nF"
+		(property "Value" "10nF"
 			(at 69.85 137.1535 0)
 			(show_name no)
@@
 			)
 		)
-		(property "MPN" "GRM1885C1H102FA01"
+		(property "MPN" "GRM1885C1H103JA01"
 			(at 67.31 135.89 0)
 			(hide yes)
@@
 			)
 		)
-		(property "Value" "1nF"
+		(property "Value" "10nF"
 			(at 69.85 77.4635 0)
 			(show_name no)
@@
 			)
 		)
-		(property "MPN" "GRM1885C1H102FA01"
+		(property "MPN" "GRM1885C1H103JA01"
 			(at 67.31 76.2 0)
 			(hide yes)
@@
 			)
 		)
-		(property "Value" "1nF"
+		(property "Value" "10nF"
 			(at 69.85 95.2435 0)
 			(show_name no)
@@
 			)
 		)
-		(property "MPN" "GRM1885C1H102FA01"
+		(property "MPN" "GRM1885C1H103JA01"
 			(at 67.31 93.98 0)
 			(hide yes)
@@
 			)
 		)
-		(property "Value" "1nF"
+		(property "Value" "10nF"
 			(at 69.85 41.9035 0)
 			(show_name no)
@@
 			)
 		)
-		(property "MPN" "GRM1885C1H102FA01"
+		(property "MPN" "GRM1885C1H103JA01"
 			(at 67.31 40.64 0)
 			(hide yes)
@@
 			)
 		)
-		(property "Value" "1nF"
+		(property "Value" "10nF"
 			(at 69.85 119.3735 0)
 			(show_name no)
@@
 			)
 		)
-		(property "MPN" "GRM1885C1H102FA01"
+		(property "MPN" "GRM1885C1H103JA01"
 			(at 67.31 118.11 0)
 			(hide yes)

Commit message: Big changes (Tim and Daniel review part 1)
Parts:
- removed F6: 100mA, APRL_Passive:Fuse_1206_3216Metric, symbol Device:Polyfuse_Small
- added F10, F12, F14, F16, F18: 100mA, APRL_Passive:Fuse_1206_3216Metric, symbol Device:Polyfuse_Small
Connections:
- net +24V: now also F10.2, F12.2, F14.2, F16.2, F18.2
- net at J14.2 (Pin_2): now also F12.1; no longer J15.2 (Pin_2)
- net at F4.1, J10.2 (Pin_2): no longer J11.2 (Pin_2)
- new net: F16.1, J16.2 (Pin_2)
- new net: F7.1, J12.2 (Pin_2)
- new net: F5.1, J11.2 (Pin_2)
- new net: F14.1, J15.2 (Pin_2)
- new net: F10.1, J13.2 (Pin_2)
- new net: F18.1, J17.2 (Pin_2)
Other:
- moved on the sheet: C29, C30, C35, C37, C38, C41, C43, C44, D10, D11, D12, D13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

Commit message: Some BoM Changes, add fabrication toolkit settings
Parts:
- C39, C40: MANUFACTURER Murata -> KEMET; MPN GRM1885C1H120JA01 -> C0603C120J5GACTU
- R20, R22, R24, R26, R28, R30, R32, R34: MANUFACTURER RESI -> Panasonic
Changed lines of the file:
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@@
 			)
 		)
-		(property "MPN" "GRM1885C1H120JA01"
+		(property "MPN" "C0603C120J5GACTU"
 			(at 223.52 132.08 0)
 			(hide yes)
@@
 			)
 		)
-		(property "MANUFACTURER" "Murata"
+		(property "MANUFACTURER" "KEMET"
 			(at 223.52 132.08 0)
 			(hide yes)
@@
 			)
 		)
-		(property "MANUFACTURER" "RESI"
+		(property "MANUFACTURER" "Panasonic"
 			(at 93.98 135.89 0)
 			(hide yes)
@@
 			)
 		)
-		(property "MPN" "GRM1885C1H120JA01"
+		(property "MPN" "C0603C120J5GACTU"
 			(at 238.76 132.08 0)
 			(hide yes)
@@
 			)
 		)
-		(property "MANUFACTURER" "Murata"
+		(property "MANUFACTURER" "KEMET"
 			(at 238.76 132.08 0)
 			(hide yes)
@@
 			)
 		)
-		(property "MANUFACTURER" "RESI"
+		(property "MANUFACTURER" "Panasonic"
 			(at 93.98 40.64 0)
 			(hide yes)
@@
 			)
 		)
-		(property "MANUFACTURER" "RESI"
+		(property "MANUFACTURER" "Panasonic"
 			(at 93.98 177.8 0)
 			(hide yes)
@@
 			)
 		)
-		(property "MANUFACTURER" "RESI"
+		(property "MANUFACTURER" "Panasonic"
 			(at 93.98 118.11 0)
 			(hide yes)
@@
 			)
 		)
-		(property "MANUFACTURER" "RESI"
+		(property "MANUFACTURER" "Panasonic"
 			(at 93.98 93.98 0)
 			(hide yes)
@@
 			)
 		)
-		(property "MANUFACTURER" "RESI"
+		(property "MANUFACTURER" "Panasonic"
 			(at 93.98 58.42 0)
 			(hide yes)
@@
 			)
 		)
-		(property "MANUFACTURER" "RESI"
+		(property "MANUFACTURER" "Panasonic"
 			(at 93.98 160.02 0)
 			(hide yes)
@@
 			)
 		)
-		(property "MANUFACTURER" "RESI"
+		(property "MANUFACTURER" "Panasonic"
 			(at 93.98 76.2 0)
 			(hide yes)
