File: ali/v2/thermocouples/thermocouples.kicad_pcb (KiCad board)
At the start: 4 copper layers, 85 x 76 mm, 151 parts, among them J1 Conn_02x01, J10 Conn_01x02, J11 Conn_01x02, J12 Conn_01x02, J13 Conn_01x02, J14 Conn_01x02, J2 Conn_01x05, J26 Vertical Ethernet, J3 USB_C_Receptacle_USB2.0_16P, J4 Conn_01x15, J5 Conn_02x09_Counter_Clockwise, J6 Screw_Terminal_01x02, J8 Conn_01x03, J9 Conn_01x02, SW1 SKRPANE010, U1 STM32H563RIV6, U14 TMP1075DSG, U17 TMP1075DSG, U18 TMP1075DSG, U19 TMP1075DSG, U2 UCC33420-Q1, U20 TMP1075DSG, U21 TMP1075DSG, U3 AP2112K-3.3, U4 TJA1462ATK, U6 ADS124S08, U7 LAN8742AI, Y1 25 MHz, Y2 25 MHz

Commit message: Small cleanups
Parts:
- removed D10, D11, D12, D13, D14, D15, D16, D17, D6, D7, D8, D9: VTVS28ASMF, Diode_SMD:D_SMF
- removed U6: ADS124S08, APRL_Package_QFN:Texas_RHB0032M_VQFN-32-1EP_5x5mm_P0.5mm_EP2.1x2.1mm_ThermalVias
- added U5: ADS124S08, APRL_Package_QFN:Texas_RHB0032M_VQFN-32-1EP_5x5mm_P0.5mm_EP2.1x2.1mm_ThermalVias, F.Cu at (133.7, 83.7)
- moved R28 2.46 mm to (119.8, 121.0)
- moved C38 2.46 mm to (124.2, 122.5)
- moved R24 2.46 mm to (122.0, 123.3)
- moved R26 2.46 mm to (122.0, 121.7)
- moved C32 2.46 mm to (122.0, 124.9)
- moved C40 2.46 mm to (122.0, 120.1)
- moved C21 1.84 mm to (149.0, 119.2), turned to -90 degrees
- moved C10 1.24 mm to (149.4, 105.8)
- moved C22 0.45 mm to (147.4, 119.2), turned to -90 degrees
Connections:
- net /ADC/AIN0 renamed Net-(U5-AIN0)
- net /ADC/AIN1 renamed Net-(U5-AIN1)
- net /ADC/AIN10 renamed Net-(U5-GPIO2/AIN10)
- net /ADC/AIN11 renamed Net-(U5-GPIO3/AIN11)
- net /ADC/AIN2 renamed Net-(U5-AIN2)
- net /ADC/AIN3 renamed Net-(U5-AIN3)
- net /ADC/AIN4 renamed Net-(U5-AIN4)
- net /ADC/AIN5 renamed Net-(U5-AIN5)
- net /ADC/AIN6 renamed Net-(U5-REFP1/AIN6)
- net /ADC/AIN7 renamed Net-(U5-REFN1/AIN7)
- net /ADC/AIN8 renamed Net-(U5-GPIO0/AIN8)
- net /ADC/AIN9 renamed Net-(U5-GPIO1/AIN9)
Routing:
- net Net-(J9-Pin_2): track 15.5 -> 9.87 mm
- net Net-(J9-Pin_1): track 8.53 -> 2.90 mm
- net Net-(J14-Pin_2): track 15.5 -> 12.3 mm
- net Net-(J13-Pin_2): track 15.5 -> 12.3 mm
- net Net-(J12-Pin_2): track 15.5 -> 12.3 mm
- net Net-(J11-Pin_2): track 15.5 -> 12.3 mm
- net Net-(J10-Pin_2): track 15.5 -> 12.3 mm
- net Net-(J10-Pin_1): track 8.53 -> 5.32 mm
- net Net-(J14-Pin_1): track 8.53 -> 5.32 mm
- net Net-(J13-Pin_1): track 8.53 -> 5.32 mm
- net Net-(J12-Pin_1): track 8.53 -> 5.32 mm
- net Net-(J11-Pin_1): track 8.53 -> 5.32 mm
- net Net-(U5-AIN1): track 42.7 -> 45.2 mm
- net Net-(U5-AIN0): track 44.0 -> 46.5 mm
- net GND: track 4.33 -> 6.49 mm, vias 379 -> 373
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
Commit message: Big changes (Tim and Daniel review part 1)
Parts:
- H1, H2, H3, H4: footprint MountingHole:MountingHole_3.2mm_M3 -> APRL_Misc:MountingHole_3.2mm_M3
- J6: footprint Connector_Phoenix_MSTB:PhoenixContact_MSTBV_2,5_2-GF-5,08_1x02_P5.08mm_Vertical_ThreadedFlange_MountHole -> APRL_Connector:PhoenixContact_MSTBV_2,5_2-GF-5,08_1x02_P5.08mm_Vertical_ThreadedFlange_MountHole
- U14, U17, U18, U19, U20, U21: footprint Package_SON:Texas_DSG0008A_WSON-8-1EP_2x2mm_P0.5mm_EP0.9x1.6mm_ThermalVias -> APRL_Package_QFN:Texas_DSG0008A_WSON-8-1EP_2x2mm_P0.5mm_EP0.9x1.6mm_ThermalVias
- moved R47 1.50 mm to (124.5, 66.8), turned to -90 degrees
- moved R46 1.41 mm to (126.3, 67.7), turned to -90 degrees
Routing:
- net +3.3V: track 158.1 -> 144.4 mm, vias 35 -> 36
- net GND: vias 373 -> 382

Commit message: Minor clearance problems
Routing:
- net /CJC Sensors/SCL: track 153.6 -> 154.6 mm
Changed lines of the file:
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@@
 	)
 	(segment
-		(start 163.3125 97.825)
-		(end 163.3125 98.925)
+		(start 155.7125 76.135)
+		(end 166.174044 76.135)
 		(width 0.3)
 		(layer "B.Cu")
@@
 	)
 	(segment
-		(start 155.7125 76.135)
-		(end 166.174044 76.135)
+		(start 162.9325 98.205)
+		(end 162.9325 100.155)
 		(width 0.3)
 		(layer "B.Cu")
@@
 	)
 	(segment
-		(start 160.5125 101.725)
-		(end 160.5125 101.925)
+		(start 166.174044 76.135)
+		(end 168.564044 78.525)
 		(width 0.3)
 		(layer "B.Cu")
@@
 	)
 	(segment
-		(start 175.4125 79.925)
-		(end 175.4125 94.125)
+		(start 161.1625 101.925)
+		(end 160.5125 101.925)
 		(width 0.3)
 		(layer "B.Cu")
@@
 	)
 	(segment
-		(start 160.5125 101.925)
-		(end 158.9125 103.525)
+		(start 164.4125 96.725)
+		(end 162.9325 98.205)
 		(width 0.3)
 		(layer "B.Cu")
@@
 	)
 	(segment
-		(start 175.4125 94.125)
-		(end 172.8125 96.725)
+		(start 175.4125 79.925)
+		(end 175.4125 94.125)
 		(width 0.3)
 		(layer "B.Cu")
@@
 	)
 	(segment
-		(start 163.3125 98.925)
-		(end 160.5125 101.725)
+		(start 175.4125 94.125)
+		(end 172.8125 96.725)
 		(width 0.3)
 		(layer "B.Cu")
@@
 	)
 	(segment
-		(start 158.9125 103.525)
-		(end 158.9125 104.325)
+		(start 160.5125 101.925)
+		(end 158.9125 103.525)
 		(width 0.3)
 		(layer "B.Cu")
@@
 	)
 	(segment
-		(start 166.174044 76.135)
-		(end 168.564044 78.525)
+		(start 162.9325 100.155)
+		(end 161.1625 101.925)
 		(width 0.3)
 		(layer "B.Cu")
@@
 	)
 	(segment
-		(start 164.4125 96.725)
-		(end 163.3125 97.825)
+		(start 158.9125 103.525)
+		(end 158.9125 104.325)
 		(width 0.3)
 		(layer "B.Cu")
@@
 	)
 	(segment
-		(start 161.3125 114.625)
-		(end 164.6125 114.625)
+		(start 160.2125 115.725)
+		(end 161.3125 114.625)
 		(width 0.15)
 		(layer "B.Cu")
@@
 	)
 	(segment
-		(start 171.7375 117.825)
-		(end 174.8125 114.75)
+		(start 167.8525 117.865)
+		(end 171.6975 117.865)
 		(width 0.15)
 		(layer "B.Cu")
@@
 	)
 	(segment
-		(start 160.2125 115.725)
-		(end 161.3125 114.625)
+		(start 171.6975 117.865)
+		(end 174.8125 114.75)
 		(width 0.15)
 		(layer "B.Cu")
@@
 	(segment
 		(start 164.6125 114.625)
-		(end 167.8125 117.825)
+		(end 167.8525 117.865)
 		(width 0.15)
 		(layer "B.Cu")
@@
 	)
 	(segment
-		(start 167.8125 117.825)
-		(end 171.7375 117.825)
+		(start 161.3125 114.625)
+		(end 164.6125 114.625)
 		(width 0.15)
 		(layer "B.Cu")
@@
 	)
 	(segment
+		(start 140.891501 70.104001)
+		(end 138.7625 67.975)
+		(width 0.15)
+		(layer "F.Cu")
+		(net "/CJC Sensors/SDA")
+	)
+	(segment
 		(start 115.3025 89.845)
 		(end 116.135 90.6775)
@@
 	)
 	(segment
+		(start 128.8325 68.425)
+		(end 126.3125 68.425)
+		(width 0.15)
+		(layer "F.Cu")
+		(net "/CJC Sensors/SDA")
+	)
+	(segment
 		(start 116.135 74.005)
 		(end 116.135 68.3475)
@@
 	)
 	(segment
-		(start 140.891501 73.225)
-		(end 140.891501 70.104001)
+		(start 111.1125 118.125)
+		(end 115.5125 118.125)
 		(width 0.15)
 		(layer "F.Cu")
@@
 	)
 	(segment
-		(start 111.1125 118.125)
-		(end 115.5125 118.125)
+		(start 126.3125 68.425)
+		(end 116.2125 68.425)
+		(width 0.15)
+		(layer "F.Cu")
+		(net "/CJC Sensors/SDA")
+	)
+	(segment
+		(start 138.7625 67.975)
+		(end 129.2825 67.975)
 		(width 0.15)
 		(layer "F.Cu")
@@
 	)
 	(segment
+		(start 116.2125 68.425)
+		(end 116.1125 68.325)
+		(width 0.15)
+		(layer "F.Cu")
+		(net "/CJC Sensors/SDA")
+	)
+	(segment
 		(start 116.135 100.3475)
 		(end 116.135 101.605)
@@
 	)
 	(segment
-		(start 139.1125 68.325)
-		(end 116.1125 68.325)
+		(start 129.2825 67.975)
+		(end 128.8325 68.425)
 		(width 0.15)
 		(layer "F.Cu")
@@
 	)
 	(segment
-		(start 140.891501 70.104001)
-		(end 139.1125 68.325)
-		(width 0.15)
-		(layer "F.Cu")
-		(net "/CJC Sensors/SDA")
-	)
-	(segment
 		(start 116.135 81.7475)
 		(end 116.135 83.205)
@@
 	)
 	(segment
+		(start 140.891501 73.225)
+		(end 140.891501 70.104001)
+		(width 0.15)
+		(layer "F.Cu")
+		(net "/CJC Sensors/SDA")
+	)
+	(segment
 		(start 109.9125 116.925)
 		(end 111.1125 118.125)
@@
 	)
 	(segment
+		(start 115.7925 67.045)
+		(end 115.3125 67.525)
+		(width 0.15)
+		(layer "F.Cu")
+		(net "/CJC Sensors/SCL")
+	)
+	(segment
 		(start 109.1125 109.115)
 		(end 109.1125 117.325)
@@
 	)
 	(segment
+		(start 142.3915 71.224999)
+		(end 142.3915 69.804)
+		(width 0.15)
+		(layer "F.Cu")
+		(net "/CJC Sensors/SCL")
+	)
+	(segment
 		(start 109.1125 90.855)
 		(end 109.1125 99.125)
@@
 	)
 	(segment
-		(start 140.1125 67.525)
-		(end 115.3125 67.525)
+		(start 128.0425 67.725)
+		(end 116.4725 67.725)
 		(width 0.15)
 		(layer "F.Cu")
@@
 	)
 	(segment
-		(start 142.3915 69.804)
-		(end 140.1125 67.525)
+		(start 109.1125 81.545)
+		(end 109.1125 89.925)
 		(width 0.15)
 		(layer "F.Cu")
@@
 	)
 	(segment
-		(start 109.1125 81.545)
-		(end 109.1125 89.925)
+		(start 115.635 110.0475)
+		(end 114.7025 109.115)
 		(width 0.15)
 		(layer "F.Cu")
@@
 	)
 	(segment
-		(start 115.635 110.0475)
-		(end 114.7025 109.115)
+		(start 116.4725 67.725)
+		(end 115.7925 67.045)
 		(width 0.15)
 		(layer "F.Cu")
@@
 	)
 	(segment
-		(start 142.3915 71.224999)
-		(end 142.3915 69.804)
+		(start 128.7225 67.045)
+		(end 128.0425 67.725)
+		(width 0.15)
+		(layer "F.Cu")
+		(net "/CJC Sensors/SCL")
+	)
+	(segment
+		(start 139.6325 67.045)
+		(end 128.7225 67.045)
 		(width 0.15)
 		(layer "F.Cu")
@@
 		(width 0.15)
 		(layer "F.Cu")
+		(net "/CJC Sensors/SCL")
+	)
+	(segment
+		(start 142.3915 69.804)
+		(end 139.6325 67.045)
+		(width 0.15)
+		(layer "F.Cu")

Commit message: more clearance
Routing:
- net Net-(U7-LED1/REGOFF): track 44.9 -> 40.0 mm
- net Net-(J26-Pad10): track 10.8 -> 14.0 mm
- net /ADC/CS: track 15.9 -> 14.4 mm
- net GND: vias 382 -> 425
