File: ali/v2/thermocouples/thermocouples.kicad_pcb (KiCad board)
At the start: 4 copper layers, 85 x 76 mm, 139 parts, among them J1 Conn_02x01, J10 Conn_01x02, J11 Conn_01x02, J12 Conn_01x02, J13 Conn_01x02, J14 Conn_01x02, J2 Conn_01x05, J26 Vertical Ethernet, J3 USB_C_Receptacle_USB2.0_16P, J4 Conn_01x15, J5 Conn_02x09_Counter_Clockwise, J6 Screw_Terminal_01x02, J8 Conn_01x03, J9 Conn_01x02, SW1 SKRPANE010, U1 STM32H563RIV6, U14 TMP1075DSG, U17 TMP1075DSG, U18 TMP1075DSG, U19 TMP1075DSG, U2 UCC33420-Q1, U20 TMP1075DSG, U21 TMP1075DSG, U3 AP2112K-3.3, U4 TJA1462ATK, U5 ADS124S08, U7 LAN8742AI, Y1 25 MHz, Y2 25 MHz

Commit message: Use 1206 on AFEs
Parts:
- C38, C39, C44, C45, C51, C52: footprint APRL_Passive:C_0603 -> APRL_Passive:C_1206
- moved C38 2.14 mm to (126.3, 122.2)
- moved R26 1.59 mm to (123.5, 121.4)
- moved C32 1.59 mm to (123.5, 124.6)
- moved C40 1.59 mm to (123.5, 119.8)
- moved R24 1.59 mm to (123.5, 123.0)
- moved R28 1.59 mm to (121.3, 120.7)
- moved R29 0.90 mm to (121.3, 102.5)
- moved R30 0.90 mm to (121.3, 111.7)
- moved R31 0.90 mm to (121.3, 93.3)
- moved R36 0.90 mm to (121.3, 84.1)
- moved R37 0.90 mm to (121.3, 74.9)
- moved C33 0.90 mm to (123.5, 115.6)
- moved C41 0.90 mm to (123.5, 110.8)
- moved C42 0.90 mm to (123.5, 106.4)
- moved C43 0.90 mm to (123.5, 97.2)
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Routing:
- net Net-(U5-AIN1): track 45.2 -> 42.7 mm
- net Net-(J9-Pin_1): track 2.90 -> 4.61 mm
- net Net-(J9-Pin_2): track 9.87 -> 11.6 mm
- net Net-(U5-AIN4): track 24.1 -> 25.8 mm
- net Net-(U5-GPIO2/AIN10): track 13.5 -> 15.0 mm
- net Net-(U5-GPIO3/AIN11): track 14.8 -> 16.2 mm
- net Net-(U5-GPIO0/AIN8): track 18.4 -> 19.8 mm
- net Net-(U5-AIN2): track 34.5 -> 35.9 mm
- net Net-(U5-REFP1/AIN6): track 16.4 -> 17.8 mm
- net +ADC_VREF: track 69.2 -> 68.1 mm
- net Net-(U5-AIN0): track 46.5 -> 45.6 mm
- net Net-(J10-Pin_1): track 5.32 -> 4.48 mm
- net Net-(J12-Pin_1): track 5.32 -> 4.48 mm
- net Net-(U5-AIN5): track 23.0 -> 23.8 mm
- net Net-(J14-Pin_1): track 5.32 -> 4.56 mm
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