File: ali/v2/thermocouples/connectivity.kicad_sch (KiCad schematic)
At the start: 27 parts, among them J26 Vertical Ethernet, J8 Conn_01x03, U4 TJA1462ATK, U7 LAN8742AI, Y2 25 MHz

Commit message: Some BoM Changes, add fabrication toolkit settings
Parts:
- R12: MPN RC0603FR-071K5L -> AC0603FR-071K5L
- R13, R14, R15, R16: MPN RC0603FR-0747RL -> AC0603FR-0747RL
- R17, R51: MPN RC0603FR-0710KL -> AC0603FR-0710KL
- R52, R53: MPN RC0603FR-07330RL -> AC0603FR-07330RL
Changed lines of the file:
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@@
 			)
 		)
-		(property "MPN" "RC0603FR-07330RL"
+		(property "MPN" "AC0603FR-07330RL"
 			(at 144.78 100.33 0)
 			(hide yes)
@@
 			)
 		)
-		(property "MPN" "RC0603FR-0747RL"
+		(property "MPN" "AC0603FR-0747RL"
 			(at 100.33 64.77 0)
 			(hide yes)
@@
 			)
 		)
-		(property "MPN" "RC0603FR-0710KL"
+		(property "MPN" "AC0603FR-0710KL"
 			(at 53.34 81.28 90)
 			(hide yes)
@@
 			)
 		)
-		(property "MPN" "RC0603FR-07330RL"
+		(property "MPN" "AC0603FR-07330RL"
 			(at 157.48 100.33 0)
 			(hide yes)
@@
 			)
 		)
-		(property "MPN" "RC0603FR-0747RL"
+		(property "MPN" "AC0603FR-0747RL"
 			(at 119.38 64.77 0)
 			(hide yes)
@@
 			)
 		)
-		(property "MPN" "RC0603FR-0710KL"
+		(property "MPN" "AC0603FR-0710KL"
 			(at 99.06 97.79 0)
 			(hide yes)
@@
 			)
 		)
-		(property "MPN" "RC0603FR-0747RL"
+		(property "MPN" "AC0603FR-0747RL"
 			(at 109.22 64.77 0)
 			(hide yes)
@@
 			)
 		)
-		(property "MPN" "RC0603FR-0747RL"
+		(property "MPN" "AC0603FR-0747RL"
 			(at 129.54 64.77 0)
 			(hide yes)
@@
 			)
 		)
-		(property "MPN" "RC0603FR-071K5L"
+		(property "MPN" "AC0603FR-071K5L"
 			(at 43.18 63.5 0)
 			(hide yes)
