File: ali/v2/thermocouples/microcontroller.kicad_sch (KiCad schematic)
At the start: 45 parts, among them J1 Conn_02x01, J2 Conn_01x05, J3 USB_C_Receptacle_USB2.0_16P, J4 Conn_01x15, J5 Conn_02x09_Counter_Clockwise, J6 Screw_Terminal_01x02, SW1 SKRPANE010, U1 STM32H563RIV6, U2 UCC33420-Q1, U3 AP2112K-3.3, Y1 25 MHz

Commit message: Big changes (Tim and Daniel review part 1)
Parts:
- J6: footprint Connector_Phoenix_MSTB:PhoenixContact_MSTBV_2,5_2-GF-5,08_1x02_P5.08mm_Vertical_ThreadedFlange_MountHole -> APRL_Connector:PhoenixContact_MSTBV_2,5_2-GF-5,08_1x02_P5.08mm_Vertical_ThreadedFlange_MountHole

Commit message: Some BoM Changes, add fabrication toolkit settings
Parts:
- J5: MANUFACTURER (none) -> Lian Xin Technology; MPN (none) -> XDFH-0254-2*9P
- R1, R2: MPN RC0603FR-075K1L -> AC0603FR-075K1L
- R3, R4, R5, R6, R7: MPN RC0603FR-0710KL -> AC0603FR-0710KL
- U3: MANUFACTURER Didoes Inc. -> Diodes Inc.
