File: ali/v2/thermocouples/analog.kicad_sch (KiCad schematic)
At the start: 60 parts, among them J10 Conn_01x02, J11 Conn_01x02, J12 Conn_01x02, J13 Conn_01x02, J14 Conn_01x02, J9 Conn_01x02, U6 ADS124S08

Commit message: Small cleanups
Parts:
- removed D10, D11, D12, D13, D14, D15, D16, D17, D6, D7, D8, D9: VTVS28ASMF, Diode_SMD:D_SMF, symbol Diode:SMF5V0A
- removed U6: ADS124S08, APRL_Package_QFN:Texas_RHB0032M_VQFN-32-1EP_5x5mm_P0.5mm_EP2.1x2.1mm_ThermalVias, symbol APRL_Analog:ADS124S08
- added U5: ADS124S08, APRL_Package_QFN:Texas_RHB0032M_VQFN-32-1EP_5x5mm_P0.5mm_EP2.1x2.1mm_ThermalVias, symbol APRL_Analog:ADS124S08
Connections:
- net +3.3V: now also U5.15 (IOVDD), U5.16 (DVDD)
- net +5V: now also U5.26 (AVDD)
- net +ADC_VREF: now also U5.23 (REFOUT)
- net CS: now also U5.9 (CS)
- net DRDY: now also U5.13 (DRDY)
- net GND: now also U5.1 (AINCOM), U5.14 (DGND), U5.17 (CLK), U5.24 (REFCOM), U5.27 (AVSS), U5.28 (AVSS-SW), U5.33 (EP)
- net MISO: now also U5.12 (DOUT/DRDY)
- net MOSI: now also U5.10 (DIN)
- net RESET: now also U5.18 (RESET)
- net SCLK: now also U5.11 (SCLK)
- net START: now also U5.8 (START/SYNC)
- net AIN0: no longer names the net of C32.1, C38.2, R24.2
- net AIN0: now also U5.7 (AIN0)
- net AIN1: no longer names the net of C38.1, C40.2, R26.2
- net AIN1: now also U5.6 (AIN1)
- net AIN10: no longer names the net of C50.1, C52.2, R41.2
- net AIN10: now also U5.20 (GPIO2/AIN10)
- net AIN11: no longer names the net of C52.1, C54.2, R43.2
- net AIN11: now also U5.19 (GPIO3/AIN11)
- net AIN2: no longer names the net of C33.1, C39.2, R25.2
- net AIN2: now also U5.5 (AIN2)
- net AIN3: no longer names the net of C39.1, C41.2, R27.2
- net AIN3: now also U5.4 (AIN3)
- net AIN4: no longer names the net of C42.1, C44.2, R32.2
- net AIN4: now also U5.3 (AIN4)
- net AIN5: no longer names the net of C44.1, C47.2, R34.2
- net AIN5: now also U5.2 (AIN5)
- net AIN6: no longer names the net of C43.1, C45.2, R33.2
- net AIN6: now also U5.32 (REFP1/AIN6)
- net AIN7: no longer names the net of C45.1, C48.2, R35.2
- net AIN7: now also U5.31 (REFN1/AIN7)
- net AIN8: no longer names the net of C49.1, C51.2, R40.2
- net AIN8: now also U5.22 (GPIO0/AIN8)
- net AIN9: no longer names the net of C51.1, C53.2, R42.2
- net AIN9: now also U5.21 (GPIO1/AIN9)
Other:
- note removed: "ADC"
- note removed: "INPUTS"
- note removed: "Should be able to handle +12/24V transients at least until the short burns itself out"
- note removed: "Still need to make this one not blocky"
- note removed: "The diodes are more for HV transients and can be removed. The actual +24V short case is handled by the series resistors, wherein the max current input per pin is 10 mA, so 24/4700 is around 5mA"
- moved on the sheet: C32, C33, C34, C35, C36, C37, C38, C39, C40, C41, C42, C43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

Commit message: Some BoM Changes, add fabrication toolkit settings
Parts:
- U5: MANUFACTURER (none) -> TI; MPN (none) -> ADS124S08IRHBT
Changed lines of the file:
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@@
+			)
+		)
+		(property "MPN" "ADS124S08IRHBT"
+			(at 179.07 111.76 0)
+			(hide yes)
+			(show_name no)
+			(do_not_autoplace no)
+			(effects
+				(font
+					(size 1.27 1.27)
+				)
+			)
+		)
+		(property "MANUFACTURER" "TI"
+			(at 179.07 111.76 0)
+			(hide yes)
+			(show_name no)
+			(do_not_autoplace no)
+			(effects
+				(font
+					(size 1.27 1.27)
+				)
 			)
 		)

Commit message: Use 1206 on AFEs
Parts:
- C38, C39, C44, C45, C51, C52: footprint APRL_Passive:C_0603 -> APRL_Passive:C_1206
Changed lines of the file:
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@@
 			)
 		)
-		(property "Footprint" "APRL_Passive:C_0603"
+		(property "Footprint" "APRL_Passive:C_1206"
 			(at 107.95 95.25 0)
 			(hide yes)
@@
 			)
 		)
-		(property "Footprint" "APRL_Passive:C_0603"
+		(property "Footprint" "APRL_Passive:C_1206"
 			(at 67.31 125.73 0)
 			(hide yes)
@@
 			)
 		)
-		(property "Footprint" "APRL_Passive:C_0603"
+		(property "Footprint" "APRL_Passive:C_1206"
 			(at 107.95 156.21 0)
 			(hide yes)
@@
 			)
 		)
-		(property "Footprint" "APRL_Passive:C_0603"
+		(property "Footprint" "APRL_Passive:C_1206"
 			(at 68.58 176.53 0)
 			(hide yes)
@@
 			)
 		)
-		(property "Footprint" "APRL_Passive:C_0603"
+		(property "Footprint" "APRL_Passive:C_1206"
 			(at 67.31 63.5 0)
 			(hide yes)
@@
 			)
 		)
-		(property "Footprint" "APRL_Passive:C_0603"
+		(property "Footprint" "APRL_Passive:C_1206"
 			(at 107.95 34.29 0)
 			(hide yes)
