File: ali/v2/loadcells/connectivity.kicad_sch (KiCad schematic)
At the start: 27 parts, among them J26 Vertical Ethernet, J8 Conn_01x03, U4 TJA1462ATK, U7 LAN8742AI, Y2 25 MHz

Commit message: Some BoM Changes, add fabrication toolkit settings
Parts:
- R12: MPN RC0603FR-071K5L -> AC0603FR-071K5L
- R13, R14, R15, R16: MPN RC0603FR-0747RL -> AC0603FR-0747RL
- R17, R51: MPN RC0603FR-0710KL -> AC0603FR-0710KL
- R52, R53: MPN RC0603FR-07330RL -> AC0603FR-07330RL
Changed lines of the file:
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@@
 			)
 		)
-		(property "MPN" "RC0603FR-0747RL"
+		(property "MPN" "AC0603FR-0747RL"
 			(at 111.76 67.31 0)
 			(hide yes)
@@
 			)
 		)
-		(property "MPN" "RC0603FR-07330RL"
+		(property "MPN" "AC0603FR-07330RL"
 			(at 147.32 102.87 0)
 			(hide yes)
@@
 			)
 		)
-		(property "MPN" "RC0603FR-0747RL"
+		(property "MPN" "AC0603FR-0747RL"
 			(at 132.08 67.31 0)
 			(hide yes)
@@
 			)
 		)
-		(property "MPN" "RC0603FR-0747RL"
+		(property "MPN" "AC0603FR-0747RL"
 			(at 121.92 67.31 0)
 			(hide yes)
@@
 			)
 		)
-		(property "MPN" "RC0603FR-071K5L"
+		(property "MPN" "AC0603FR-071K5L"
 			(at 45.72 66.04 0)
 			(hide yes)
@@
 			)
 		)
-		(property "MPN" "RC0603FR-0710KL"
+		(property "MPN" "AC0603FR-0710KL"
 			(at 55.88 83.82 90)
 			(hide yes)
@@
 			)
 		)
-		(property "MPN" "RC0603FR-0747RL"
+		(property "MPN" "AC0603FR-0747RL"
 			(at 102.87 67.31 0)
 			(hide yes)
@@
 			)
 		)
-		(property "MPN" "RC0603FR-0710KL"
+		(property "MPN" "AC0603FR-0710KL"
 			(at 101.6 100.33 0)
 			(hide yes)
@@
 			)
 		)
-		(property "MPN" "RC0603FR-07330RL"
+		(property "MPN" "AC0603FR-07330RL"
 			(at 160.02 102.87 0)
 			(hide yes)
