File: ali/v2/loadcells/load-cell.kicad_pcb (KiCad board)
At the start: 4 copper layers, 85 x 76 mm, 113 parts, among them J1 Conn_02x01, J10 Conn_01x04, J11 Conn_01x04, J12 Conn_01x04, J2 Conn_01x05, J26 Vertical Ethernet, J3 USB_C_Receptacle_USB2.0_16P, J4 Conn_01x15, J5 Conn_02x09_Counter_Clockwise, J6 Screw_Terminal_01x02, J8 Conn_01x03, J9 Conn_01x04, SW1 SKRPANE010, U1 STM32H563RIV6, U2 AP2112K-3.3, U4 TJA1462ATK, U6 ADS124S08, U7 LAN8742AI, Y1 25 MHz, Y2 25 MHz

Commit message: Small cleanups
Parts:
- D10, D11, D12, D13, D6, D7, D8, D9: moved to F.Cu
- moved D12 5.37 mm to (112.3, 123.9)
- moved D11 5.36 mm to (112.3, 105.1)
- moved D10 5.36 mm to (112.3, 110.2)
- moved D13 5.36 mm to (112.3, 118.9)
- moved D9 5.17 mm to (112.1, 91.4)
- moved D8 5.16 mm to (112.1, 96.4)
- moved D7 4.57 mm to (111.5, 77.1)
- moved D6 4.57 mm to (111.5, 82.4)
- moved C63 3.17 mm to (119.6, 82.5)
- moved C21 2.06 mm to (149.4, 119.1), turned to -90 degrees
- moved C10 1.24 mm to (149.5, 105.7)
- moved C24 0.30 mm to (147.8, 119.1), turned to -90 degrees
Connections:
- net /Microcontroller/USER_LED_1 renamed Net-(U1-PD12)
- net /Microcontroller/USER_LED_2 renamed Net-(U1-PC6)
- net /Microcontroller/USER_LED_3 renamed Net-(U1-PC7)
- C34 pad 1: Net-(U6-GPIO0/AIN8) -> Net-(D6-A1)
- C35 pad 1: Net-(U6-GPIO1/AIN9) -> Net-(D7-A1)
- C35 pad 2: Net-(U6-GPIO0/AIN8) -> Net-(D6-A1)
- C36 pad 2: Net-(U6-GPIO1/AIN9) -> Net-(D7-A1)
- C37 pad 1: Net-(U6-AIN4) -> Net-(D8-A1)
- C38 pad 2: Net-(U6-AIN5) -> Net-(D9-A1)
- C39 pad 1: Net-(U6-AIN5) -> Net-(D9-A1)
- C39 pad 2: Net-(U6-AIN4) -> Net-(D8-A1)
- C42 pad 1: Net-(U6-AIN2) -> Net-(D10-A1)
- C43 pad 2: Net-(U6-AIN3) -> Net-(D11-A1)
- C44 pad 1: Net-(U6-AIN3) -> Net-(D11-A1)
- C44 pad 2: Net-(U6-AIN2) -> Net-(D10-A1)
- C45 pad 1: Net-(U6-AIN0) -> Net-(D12-A1)
- C46 pad 2: Net-(U6-AIN1) -> Net-(D13-A1)
- C47 pad 1: Net-(U6-AIN1) -> Net-(D13-A1)
- C47 pad 2: Net-(U6-AIN0) -> Net-(D12-A1)
- J10 pad 2: Net-(D8-A1) -> Net-(J10-Pin_2)
- J10 pad 3: Net-(D9-A1) -> Net-(J10-Pin_3)
- J11 pad 2: Net-(D10-A1) -> Net-(J11-Pin_2)
- J11 pad 3: Net-(D11-A1) -> Net-(J11-Pin_3)
- J12 pad 2: Net-(D12-A1) -> Net-(J12-Pin_2)
- J12 pad 3: Net-(D13-A1) -> Net-(J12-Pin_3)
- J9 pad 2: Net-(D6-A1) -> Net-(J9-Pin_2)
- J9 pad 3: Net-(D7-A1) -> Net-(J9-Pin_3)
- R22 pad 1: Net-(D6-A1) -> Net-(J9-Pin_2)
- R22 pad 2: Net-(U6-GPIO0/AIN8) -> Net-(D6-A1)
- R23 pad 1: Net-(D7-A1) -> Net-(J9-Pin_3)
- R23 pad 2: Net-(U6-GPIO1/AIN9) -> Net-(D7-A1)
- R24 pad 1: Net-(D8-A1) -> Net-(J10-Pin_2)
- R24 pad 2: Net-(U6-AIN4) -> Net-(D8-A1)
- R25 pad 1: Net-(D9-A1) -> Net-(J10-Pin_3)
- R25 pad 2: Net-(U6-AIN5) -> Net-(D9-A1)
- R26 pad 1: Net-(D10-A1) -> Net-(J11-Pin_2)
- R26 pad 2: Net-(U6-AIN2) -> Net-(D10-A1)
- R27 pad 1: Net-(D11-A1) -> Net-(J11-Pin_3)
- R27 pad 2: Net-(U6-AIN3) -> Net-(D11-A1)
- R28 pad 1: Net-(D12-A1) -> Net-(J12-Pin_2)
- R28 pad 2: Net-(U6-AIN0) -> Net-(D12-A1)
- R29 pad 1: Net-(D13-A1) -> Net-(J12-Pin_3)
- R29 pad 2: Net-(U6-AIN1) -> Net-(D13-A1)
- U6 pad 2: Net-(U6-AIN5) -> Net-(D9-A1)
- U6 pad 21: Net-(U6-GPIO1/AIN9) -> Net-(D7-A1)
- U6 pad 22: Net-(U6-GPIO0/AIN8) -> Net-(D6-A1)
- U6 pad 3: Net-(U6-AIN4) -> Net-(D8-A1)
- U6 pad 4: Net-(U6-AIN3) -> Net-(D11-A1)
- U6 pad 5: Net-(U6-AIN2) -> Net-(D10-A1)
- U6 pad 6: Net-(U6-AIN1) -> Net-(D13-A1)
- U6 pad 7: Net-(U6-AIN0) -> Net-(D12-A1)
Routing:
- net Net-(U6-AIN0): track 50.2 -> 0.00 mm
- net Net-(U6-AIN1): track 48.4 -> 0.00 mm
- net Net-(D13-A1): track 4.84 -> 48.4 mm
- net Net-(D12-A1): track 9.33 -> 50.2 mm
- net Net-(U6-AIN2): track 35.5 -> 0.00 mm
- net Net-(U6-AIN3): track 33.8 -> 0.00 mm
- net Net-(D11-A1): track 4.84 -> 33.8 mm
- net Net-(D10-A1): track 9.33 -> 35.5 mm
- net Net-(U6-AIN4): track 21.1 -> 0.00 mm
- net Net-(U6-GPIO1/AIN9): track 19.6 -> 0.00 mm
- net Net-(U6-AIN5): track 19.3 -> 0.00 mm
- net Net-(U6-GPIO0/AIN8): track 18.8 -> 0.00 mm
- net Net-(D7-A1): track 4.84 -> 19.6 mm
- net Net-(D9-A1): track 4.84 -> 19.3 mm
- net Net-(D8-A1): track 9.33 -> 21.1 mm
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
Commit message: Big changes (Tim and Daniel review part 1)
Parts:
- removed D10, D11, D12, D13, D6, D7, D8, D9: VTVS28ASMF, Diode_SMD:D_SMF
- added C49: 1nF, APRL_Passive:C_0603, F.Cu at (115.1, 82.4)
- added C50: 10nF, APRL_Passive:C_0603, F.Cu at (117.3, 83.2)
- added R31: 4.7k, APRL_Passive:R_0603, F.Cu at (116.5, 80.8)
- C1, C6: moved to F.Cu
- C48: value 10nF -> 1nF
- H1, H2, H3, H4: footprint MountingHole:MountingHole_3.2mm_M3 -> APRL_Misc:MountingHole_3.2mm_M3
- J6: footprint Connector_Phoenix_MSTB:PhoenixContact_MSTBV_2,5_2-GF-5,08_1x02_P5.08mm_Vertical_ThreadedFlange_MountHole -> APRL_Connector:PhoenixContact_MSTBV_2,5_2-GF-5,08_1x02_P5.08mm_Vertical_ThreadedFlange_MountHole
- R30: value 1k -> 4.7k
- moved J6 59.2 mm to (113.4, 69.7), turned to 0 degrees
- moved F2 49.6 mm to (117.5, 75.0), turned to 180 degrees
- moved C1 3.41 mm to (152.7, 94.3), turned to 90 degrees
- moved R30 2.82 mm to (116.5, 85.6)
- moved C48 2.26 mm to (115.1, 84.0), turned to 180 degrees
- moved C6 2.04 mm to (151.1, 94.3), turned to 90 degrees
- moved C11 1.07 mm to (141.9, 92.6)
- moved R18 0.10 mm to (149.9, 119.3)
Connections:
- C48 pad 1: GND -> Net-(U6-REFP0)
- C48 pad 2: Net-(U6-REFP0) -> GND
- J4 pad 13: /Microcontroller/PC12 -> /Microcontroller/PC11
- J5 pad 15: /Microcontroller/PA4 -> /Microcontroller/PA5
- U1 pad 20: /Microcontroller/PA4 -> unconnected-(U1-PA4-Pad20)
- U1 pad 21: /ADC/SCLK -> /Microcontroller/PA5
- U1 pad 55: unconnected-(U1-PC11-Pad55) -> /Microcontroller/PC11
- U1 pad 56: /Microcontroller/PC12 -> /ADC/DRDY
- U1 pad 57: /ADC/DRDY -> /ADC/SCLK
- U6 pad 29: GND -> Net-(U6-REFN0)
Routing:
- net /Microcontroller/PA5: track 0.00 -> 41.2 mm, vias 0 -> 2
- net /Microcontroller/PA4: track 40.9 -> 0.00 mm, vias 2 -> 0
- net /Microcontroller/PC11: track 0.00 -> 28.4 mm, vias 0 -> 3
- net /Microcontroller/PC12: track 25.1 -> 0.00 mm
- net /ADC/SCLK: track 67.0 -> 43.3 mm
- net +5V: track 27.0 -> 45.1 mm, vias 16 -> 25
- net Net-(U6-REFP0): track 0.00 -> 5.82 mm
- net Net-(U6-REFN0): track 0.00 -> 5.31 mm
- net GND: track 7.71 -> 10.3 mm, vias 330 -> 362
- net /Microcontroller/SWCLK: track 19.1 -> 20.8 mm
- net Net-(C11-Pad1): track 1.61 -> 2.42 mm
- net Net-(U6-GPIO0/AIN8): track 18.8 -> 18.3 mm
- net Net-(U6-GPIO1/AIN9): track 19.6 -> 19.0 mm
- net /ADC/DRDY: track 31.7 -> 32.1 mm, vias 4 -> 2
- removed copper zone on F.Cu, net Net-(U6-REFP0)

Commit message: Minor clearance problems
Routing:
- net +5V: track 45.1 -> 86.6 mm
- net GND: vias 362 -> 361

Commit message: more clearance
Changed lines of the file:
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@@
 	)
 	(segment
-		(start 141.6725 93.305)
-		(end 142.0075 93.64)
+		(start 142.006912 93.477355)
+		(end 142.037312 93.507755)
 		(width 0.25)
 		(layer "F.Cu")
@@
 	)
 	(segment
-		(start 142.520673 93.64)
-		(end 142.9125 94.031827)
-		(width 0.25)
+		(start 169.699099 105.425)
+		(end 171.0125 105.425)
+		(width 0.3)
 		(layer "F.Cu")
 		(net "GND")
 	)
 	(segment
-		(start 169.699099 105.425)
-		(end 171.0125 105.425)
-		(width 0.3)
+		(start 142.037312 93.507755)
+		(end 142.388428 93.507755)
+		(width 0.25)
 		(layer "F.Cu")
 		(net "GND")
@@
 	)
 	(segment
-		(start 159.3125 76.315)
-		(end 158.0025 76.315)
-		(width 0.3)
+		(start 142.388428 93.507755)
+		(end 142.9125 94.031827)
+		(width 0.25)
 		(layer "F.Cu")
 		(net "GND")
 	)
 	(segment
-		(start 142.9125 94.031827)
-		(end 142.9125 95.0375)
-		(width 0.25)
+		(start 159.3125 76.315)
+		(end 158.0025 76.315)
+		(width 0.3)
 		(layer "F.Cu")
 		(net "GND")
@@
 	)
 	(segment
-		(start 142.0075 93.64)
-		(end 142.520673 93.64)
-		(width 0.25)
-		(layer "F.Cu")
-		(net "GND")
-	)
-	(segment
-		(start 141.6725 93.295)
-		(end 141.6725 93.305)
+		(start 142.9125 94.031827)
+		(end 142.9125 95.0375)
 		(width 0.25)
 		(layer "F.Cu")
@@
 	)
 	(via
-		(at 141.6725 93.295)
+		(at 142.006912 93.477355)
 		(size 0.6)
 		(drill 0.3)
@@
 		)
 		(min_thickness 0.15)
-		(fill yes
+		(fill
 			(thermal_gap 0.5)
 			(thermal_bridge_width 0.5)
@@
 		(polygon
 			(pts
-				(xy 160.1125 79.718008) (xy 160.1125 77.276588) (xy 160.9125 76.476588) (xy 160.9125 75.918008)
-				(xy 162.6125 75.918008) (xy 162.6125 76.568008) (xy 163.4125 77.368008) (xy 163.4125 79.718008)
-				(xy 164.0125 79.718008) (xy 164.0125 77.168008) (xy 163.2125 76.368008) (xy 163.2125 74.825) (xy 153.9125 74.825)
+				(xy 159.8825 79.718008) (xy 159.8825 77.506588) (xy 160.9125 76.476588) (xy 160.9125 75.918008)
+				(xy 162.6125 75.918008) (xy 162.6125 76.568008) (xy 163.5225 77.478008) (xy 163.5225 79.718008)
+				(xy 163.8325 79.718008) (xy 163.8325 76.988008) (xy 163.2125 76.368008) (xy 163.2125 74.825) (xy 153.9125 74.825)
 				(xy 153.9125 77.218008) (xy 154.9125 77.218008) (xy 154.9125 75.618008) (xy 160.1125 75.618008)
-				(xy 160.112182 76.598716) (xy 159.5125 77.198009) (xy 159.5125 79.718008)
+				(xy 160.112182 76.598716) (xy 159.5725 77.138048) (xy 159.5725 79.718008)
 			)
 		)
