File: ali/v2/loadcells/microcontroller.kicad_sch (KiCad schematic)
At the start: 41 parts, among them J1 Conn_02x01, J2 Conn_01x05, J3 USB_C_Receptacle_USB2.0_16P, J4 Conn_01x15, J5 Conn_02x09_Counter_Clockwise, J6 Screw_Terminal_01x02, SW1 SKRPANE010, U1 STM32H563RIV6, U2 AP2112K-3.3, Y1 25 MHz

Commit message: Big changes (Tim and Daniel review part 1)
Parts:
- J6: footprint Connector_Phoenix_MSTB:PhoenixContact_MSTBV_2,5_2-GF-5,08_1x02_P5.08mm_Vertical_ThreadedFlange_MountHole -> APRL_Connector:PhoenixContact_MSTBV_2,5_2-GF-5,08_1x02_P5.08mm_Vertical_ThreadedFlange_MountHole
Connections:
- net ADC_DRDY: now also U1.56 (PC12); no longer U1.57 (PB3(JTDO)
- net ADC_SCLK: now also U1.57 (PB3(JTDO); no longer U1.21 (PA5)
- net PC11: now reaches U1.55 (PC11)
- net PC11: now also J4.13 (Pin_13)
- net PA4: no longer names the net of U1.20 (PA4)
- net PA4: no longer J5.15 (Pin_15)
- removed net PC12: J4.13 (Pin_13), U1.56 (PC12)
- new net PA5: J5.15 (Pin_15), U1.21 (PA5)

Commit message: Some BoM Changes, add fabrication toolkit settings
Parts:
- J5: MANUFACTURER (none) -> Lian Xin Technology; MPN (none) -> XDFH-0254-2*9P
- R1, R2: MPN RC0603FR-075K1L -> AC0603FR-075K1L
- R3, R4, R5, R6, R8: MPN RC0603FR-0710KL -> AC0603FR-0710KL
- U2: MANUFACTURER Didoes Inc. -> Diodes Inc.
