File: ali/v2/valvedrivers/connectivity.kicad_sch (KiCad schematic)
At the start: 27 parts, among them J8 Vertical Ethernet, J9 Conn_01x03, U5 LAN8742AI, U6 TJA1462ATK, Y2 25 MHz

Commit message: Some BoM Changes, add fabrication toolkit settings
Parts:
- R13: MPN RC0603FR-071K5L -> AC0603FR-071K5L
- R14, R15, R16, R17: MPN RC0603FR-0747RL -> AC0603FR-0747RL
- R18, R20: MPN RC0603FR-0710KL -> AC0603FR-0710KL
- R21, R22: MPN RC0603FR-07330RL -> AC0603FR-07330RL
Changed lines of the file:
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@@
 			)
 		)
-		(property "MPN" "RC0603FR-07330RL"
+		(property "MPN" "AC0603FR-07330RL"
 			(at 144.78 104.14 0)
 			(hide yes)
@@
 			)
 		)
-		(property "MPN" "RC0603FR-07330RL"
+		(property "MPN" "AC0603FR-07330RL"
 			(at 157.48 104.14 0)
 			(hide yes)
@@
 			)
 		)
-		(property "MPN" "RC0603FR-0747RL"
+		(property "MPN" "AC0603FR-0747RL"
 			(at 100.33 68.58 0)
 			(hide yes)
@@
 			)
 		)
-		(property "MPN" "RC0603FR-0710KL"
+		(property "MPN" "AC0603FR-0710KL"
 			(at 53.34 85.09 90)
 			(hide yes)
@@
 			)
 		)
-		(property "MPN" "RC0603FR-0747RL"
+		(property "MPN" "AC0603FR-0747RL"
 			(at 129.54 68.58 0)
 			(hide yes)
@@
 			)
 		)
-		(property "MPN" "RC0603FR-0747RL"
+		(property "MPN" "AC0603FR-0747RL"
 			(at 109.22 68.58 0)
 			(hide yes)
@@
 			)
 		)
-		(property "MPN" "RC0603FR-0710KL"
+		(property "MPN" "AC0603FR-0710KL"
 			(at 99.06 101.6 0)
 			(hide yes)
@@
 			)
 		)
-		(property "MPN" "RC0603FR-071K5L"
+		(property "MPN" "AC0603FR-071K5L"
 			(at 43.18 67.31 0)
 			(hide yes)
@@
 			)
 		)
-		(property "MPN" "RC0603FR-0747RL"
+		(property "MPN" "AC0603FR-0747RL"
 			(at 119.38 68.58 0)
 			(hide yes)
