File: ali/v2/valvedrivers/drivers.kicad_sch (KiCad schematic)
At the start: 40 parts, among them J10 Conn_01x02, J11 Conn_01x02, J12 Conn_01x02, J13 Conn_01x02, J14 Conn_01x02, J15 Conn_01x02, J16 Conn_01x02, J17 Conn_01x02, U7 SN74CBTLV3245A, U8 IPS4140HQ, U9 IPS4140HQ

Commit message: Some BoM Changes, add fabrication toolkit settings
Parts:
- C29, C36: MANUFACTURER Yageo -> KEMET
- R24, R25, R26, R27, R28, R29, R30, R31, R32, R33, R34, R35, R36, R37, R38, R39: MPN RC0603FR-0710KL -> AC0603FR-0710KL
Changed lines of the file:
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@@
 			)
 		)
-		(property "MPN" "RC0603FR-0710KL"
+		(property "MPN" "AC0603FR-0710KL"
 			(at 116.84 60.96 0)
 			(hide yes)
@@
 			)
 		)
-		(property "MPN" "RC0603FR-0710KL"
+		(property "MPN" "AC0603FR-0710KL"
 			(at 180.34 40.64 0)
 			(hide yes)
@@
 			)
 		)
-		(property "MPN" "RC0603FR-0710KL"
+		(property "MPN" "AC0603FR-0710KL"
 			(at 107.95 124.46 0)
 			(hide yes)
@@
 			)
 		)
-		(property "MPN" "RC0603FR-0710KL"
+		(property "MPN" "AC0603FR-0710KL"
 			(at 125.73 60.96 0)
 			(hide yes)
@@
 			)
 		)
-		(property "MANUFACTURER" "Yageo"
+		(property "MANUFACTURER" "KEMET"
 			(at 190.5 93.98 0)
 			(hide yes)
@@
 			)
 		)
-		(property "MPN" "RC0603FR-0710KL"
+		(property "MPN" "AC0603FR-0710KL"
 			(at 99.06 60.96 0)
 			(hide yes)
@@
 			)
 		)
-		(property "MANUFACTURER" "Yageo"
+		(property "MANUFACTURER" "KEMET"
 			(at 190.5 31.75 0)
 			(hide yes)
@@
 			)
 		)
-		(property "MPN" "RC0603FR-0710KL"
+		(property "MPN" "AC0603FR-0710KL"
 			(at 162.56 40.64 0)
 			(hide yes)
@@
 			)
 		)
-		(property "MPN" "RC0603FR-0710KL"
+		(property "MPN" "AC0603FR-0710KL"
 			(at 171.45 40.64 0)
 			(hide yes)
@@
 			)
 		)
-		(property "MPN" "RC0603FR-0710KL"
+		(property "MPN" "AC0603FR-0710KL"
 			(at 116.84 124.46 0)
 			(hide yes)
@@
 			)
 		)
-		(property "MPN" "RC0603FR-0710KL"
+		(property "MPN" "AC0603FR-0710KL"
 			(at 153.67 102.87 0)
 			(hide yes)
@@
 			)
 		)
-		(property "MPN" "RC0603FR-0710KL"
+		(property "MPN" "AC0603FR-0710KL"
 			(at 99.06 124.46 0)
 			(hide yes)
@@
 			)
 		)
-		(property "MPN" "RC0603FR-0710KL"
+		(property "MPN" "AC0603FR-0710KL"
 			(at 107.95 60.96 0)
 			(hide yes)
@@
 			)
 		)
-		(property "MPN" "RC0603FR-0710KL"
+		(property "MPN" "AC0603FR-0710KL"
 			(at 162.56 102.87 0)
 			(hide yes)
@@
 			)
 		)
-		(property "MPN" "RC0603FR-0710KL"
+		(property "MPN" "AC0603FR-0710KL"
 			(at 153.67 40.64 0)
 			(hide yes)
@@
 			)
 		)
-		(property "MPN" "RC0603FR-0710KL"
+		(property "MPN" "AC0603FR-0710KL"
 			(at 171.45 102.87 0)
 			(hide yes)
@@
 			)
 		)
-		(property "MPN" "RC0603FR-0710KL"
+		(property "MPN" "AC0603FR-0710KL"
 			(at 125.73 124.46 0)
 			(hide yes)
@@
 			)
 		)
-		(property "MPN" "RC0603FR-0710KL"
+		(property "MPN" "AC0603FR-0710KL"
 			(at 180.34 102.87 0)
 			(hide yes)
