File: ali/v2/valvedrivers/drivers2.kicad_sch (KiCad schematic)
At the start: 21 parts, among them J18 Conn_01x02, J19 Conn_01x02, J20 Conn_01x02, J21 Conn_01x02, U10 SN74CBTLV3245A, U11 IPS4140HQ

Commit message: Some BoM Changes, add fabrication toolkit settings
Parts:
- C42: MANUFACTURER Yageo -> KEMET
- R40, R41, R42, R43, R44, R45, R46, R47: MPN RC0603FR-0710KL -> AC0603FR-0710KL
Changed lines of the file:
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@@
 			)
 		)
-		(property "MPN" "RC0603FR-0710KL"
+		(property "MPN" "AC0603FR-0710KL"
 			(at 116.84 86.36 0)
 			(hide yes)
@@
 			)
 		)
-		(property "MANUFACTURER" "Yageo"
+		(property "MANUFACTURER" "KEMET"
 			(at 153.67 77.47 0)
 			(hide yes)
@@
 			)
 		)
-		(property "MPN" "RC0603FR-0710KL"
+		(property "MPN" "AC0603FR-0710KL"
 			(at 134.62 86.36 0)
 			(hide yes)
@@
 			)
 		)
-		(property "MPN" "RC0603FR-0710KL"
+		(property "MPN" "AC0603FR-0710KL"
 			(at 121.92 123.19 0)
 			(hide yes)
@@
 			)
 		)
-		(property "MPN" "RC0603FR-0710KL"
+		(property "MPN" "AC0603FR-0710KL"
 			(at 113.03 123.19 0)
 			(hide yes)
@@
 			)
 		)
-		(property "MPN" "RC0603FR-0710KL"
+		(property "MPN" "AC0603FR-0710KL"
 			(at 139.7 123.19 0)
 			(hide yes)
@@
 			)
 		)
-		(property "MPN" "RC0603FR-0710KL"
+		(property "MPN" "AC0603FR-0710KL"
 			(at 125.73 86.36 0)
 			(hide yes)
@@
 			)
 		)
-		(property "MPN" "RC0603FR-0710KL"
+		(property "MPN" "AC0603FR-0710KL"
 			(at 130.81 123.19 0)
 			(hide yes)
@@
 			)
 		)
-		(property "MPN" "RC0603FR-0710KL"
+		(property "MPN" "AC0603FR-0710KL"
 			(at 143.51 86.36 0)
 			(hide yes)
