File: ali/v2/valvedrivers/valvedrivers.kicad_pcb (KiCad board)
At the start: 4 copper layers, 85 x 76 mm, 145 parts, among them J1 Conn_02x01, J10 Conn_01x02, J11 Conn_01x02, J12 Conn_01x02, J13 Conn_01x02, J14 Conn_01x02, J15 Conn_01x02, J16 Conn_01x02, J17 Conn_01x02, J18 Conn_01x02, J19 Conn_01x02, J2 Conn_01x05, J20 Conn_01x02, J21 Conn_01x02, J3 USB_C_Receptacle_USB2.0_16P, J4 Screw_Terminal_01x02, J5 Screw_Terminal_01x02, J6 Screw_Terminal_01x02, J7 Conn_01x05, J8 Vertical Ethernet, J9 Conn_01x03, SW1 SKRPANE010, U1 STM32H563RIV6, U10 SN74CBTLV3245A, U11 IPS4140HQ, U2 LTV-816S, U3 AP2112K-3.3, U4 LTV-816S, U5 LAN8742AI, U6 TJA1462ATK, U7 SN74CBTLV3245A, U8 IPS4140HQ, U9 IPS4140HQ, Y1 25 MHz, Y2 25 MHz

Commit message: Small cleanups
Parts:
- moved C18 1.98 mm to (149.3, 119.1), turned to -90 degrees
- moved C10 0.92 mm to (149.2, 105.6)
- moved C19 0.32 mm to (147.7, 119.1), turned to -90 degrees
- moved C25 0.15 mm to (144.8, 115.2)
Routing:
- net +5V: track 5.23 -> 29.4 mm, vias 8 -> 4
- net GND: track 9.17 -> 12.1 mm, vias 357 -> 355
- net /Connectivity/ETH_TXD0: track 46.9 -> 47.9 mm
- net Net-(C10-Pad1): track 1.86 -> 2.82 mm
- net /Microcontroller/~{RST}: track 62.1 -> 62.6 mm
- net /Connectivity/ETH_TXD1: track 54.3 -> 54.8 mm
- net +3.3V: track 123.1 -> 123.3 mm, vias 36 -> 34
- removed copper zone on B.Cu, net +5V

Commit message: Big changes (Tim and Daniel review part 1)
Parts:
- H1, H2, H3, H4: footprint MountingHole:MountingHole_3.2mm_M3 -> APRL_Misc:MountingHole_3.2mm_M3
- J4, J5, J6: footprint Connector_Phoenix_MSTB:PhoenixContact_MSTBV_2,5_2-GF-5,08_1x02_P5.08mm_Vertical_ThreadedFlange_MountHole -> APRL_Connector:PhoenixContact_MSTBV_2,5_2-GF-5,08_1x02_P5.08mm_Vertical_ThreadedFlange_MountHole
- moved C27 0.67 mm to (159.9, 103.7)
Routing:
- net +5V: track 29.4 -> 24.7 mm, vias 4 -> 10
- net GND: track 12.1 -> 13.9 mm, vias 355 -> 360
- added copper zone on B.Cu, net +5V

Commit message: Minor clearance problems
Parts:
- moved J2 0.69 mm to (165.1, 97.2)
- moved F4 0.53 mm to (160.9, 68.6)
- moved C48 0.30 mm to (130.9, 135.8)
- moved C33 0.15 mm to (99.7, 83.7)
- moved C32 0.13 mm to (99.7, 76.4)
Routing:
- net /Microcontroller/SWCLK: track 17.0 -> 17.7 mm
- net GND: vias 360 -> 359
