File: kicadlibs/templates/ali_v2/connectivity.kicad_sch (KiCad schematic)
At the start: 27 parts, among them J7 Conn_01x03, J8 Vertical Ethernet, U3 TJA1462ATK, U4 LAN8742AI, Y2 25 MHz

Commit message: Some BoM Changes, add fabrication toolkit settings
Parts:
- R10, R11, R12, R13: MPN RC0603FR-0747RL -> AC0603FR-0747RL
- R14, R16: MPN RC0603FR-0710KL -> AC0603FR-0710KL
- R17, R18: MPN RC0603FR-07330RL -> AC0603FR-07330RL
- R9: MPN RC0603FR-071K5L -> AC0603FR-071K5L
Changed lines of the file:
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@@
 			)
 		)
-		(property "MPN" "RC0603FR-0747RL"
+		(property "MPN" "AC0603FR-0747RL"
 			(at 100.33 68.58 0)
 			(hide yes)
@@
 			)
 		)
-		(property "MPN" "RC0603FR-0710KL"
+		(property "MPN" "AC0603FR-0710KL"
 			(at 53.34 85.09 90)
 			(hide yes)
@@
 			)
 		)
-		(property "MPN" "RC0603FR-0747RL"
+		(property "MPN" "AC0603FR-0747RL"
 			(at 134.62 68.58 0)
 			(hide yes)
@@
 			)
 		)
-		(property "MPN" "RC0603FR-0747RL"
+		(property "MPN" "AC0603FR-0747RL"
 			(at 111.76 68.58 0)
 			(hide yes)
@@
 			)
 		)
-		(property "MPN" "RC0603FR-07330RL"
+		(property "MPN" "AC0603FR-07330RL"
 			(at 229.87 120.65 0)
 			(hide yes)
@@
 			)
 		)
-		(property "MPN" "RC0603FR-0710KL"
+		(property "MPN" "AC0603FR-0710KL"
 			(at 99.06 102.87 0)
 			(hide yes)
@@
 			)
 		)
-		(property "MPN" "RC0603FR-071K5L"
+		(property "MPN" "AC0603FR-071K5L"
 			(at 43.18 67.31 0)
 			(hide yes)
@@
 			)
 		)
-		(property "MPN" "RC0603FR-07330RL"
+		(property "MPN" "AC0603FR-07330RL"
 			(at 220.98 130.81 0)
 			(hide yes)
@@
 			)
 		)
-		(property "MPN" "RC0603FR-0747RL"
+		(property "MPN" "AC0603FR-0747RL"
 			(at 123.19 68.58 0)
 			(hide yes)
