File: ali/v2/isospi-transceiver/isospi.kicad_sch (KiCad schematic)
At the start: 19 parts, among them J4 Conn_01x06, U5 ADBMS6822, U6 UCC33420-Q1

Commit message: Some BoM Changes, add fabrication toolkit settings
Parts:
- J4: MANUFACTURER (none) -> Molex; MPN (none) -> 503159-0601
- R19: MPN (none) -> AC0603FR-07100RL
- R20: MPN (none) -> AC0603FR-07100KL
- TR1: MANUFACTURER (none) -> Pulse Electronics; MPN (none) -> HX1188NLT
- U5: MANUFACTURER (none) -> Analog Devices; MPN (none) -> ADBMS6822CCSZ
Changed lines of the file:
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@@
+			)
+		)
+		(property "MPN" "503159-0601"
+			(at 257.81 66.04 0)
+			(hide yes)
+			(show_name no)
+			(do_not_autoplace no)
+			(effects
+				(font
+					(size 1.27 1.27)
+				)
+			)
+		)
+		(property "MANUFACTURER" "Molex"
+			(at 257.81 66.04 0)
+			(hide yes)
+			(show_name no)
+			(do_not_autoplace no)
+			(effects
+				(font
+					(size 1.27 1.27)
+				)
 			)
 		)
@@
 			)
 		)
-		(property "MPN" ""
+		(property "MPN" "AC0603FR-07100KL"
 			(at 120.65 73.66 0)
 			(hide yes)
@@
 		)
 		(property "Description" "10/100BASE-TX single port 1:1 transformer with CM choke, 1650 Vrms, SO-16 7.11x12.7mm; isoSPI per LTC6820 Table 7"
+			(at 218.44 60.96 0)
+			(hide yes)
+			(show_name no)
+			(do_not_autoplace no)
+			(effects
+				(font
+					(size 1.27 1.27)
+				)
+			)
+		)
+		(property "MPN" "HX1188NLT"
+			(at 218.44 60.96 0)
+			(hide yes)
+			(show_name no)
+			(do_not_autoplace no)
+			(effects
+				(font
+					(size 1.27 1.27)
+				)
+			)
+		)
+		(property "MANUFACTURER" "Pulse Electronics"
 			(at 218.44 60.96 0)
 			(hide yes)
@@
 			)
 		)
+		(property "MPN" "ADBMS6822CCSZ"
+			(at 100.33 60.96 0)
+			(hide yes)
+			(show_name no)
+			(do_not_autoplace no)
+			(effects
+				(font
+					(size 1.27 1.27)
+				)
+			)
+		)
+		(property "MANUFACTURER" "Analog Devices"
+			(at 100.33 60.96 0)
+			(hide yes)
+			(show_name no)
+			(do_not_autoplace no)
+			(effects
+				(font
+					(size 1.27 1.27)
+				)
+			)
+		)
 		(pin "8"
 		)
@@
 			)
 		)
-		(property "MPN" ""
+		(property "MPN" "AC0603FR-07100RL"
 			(at 165.1 55.88 0)
 			(hide yes)
@@
 			(at 100.33 115.57 0)
 			(hide yes)
+			(show_name no)
+			(do_not_autoplace no)
+			(effects
+				(font
+					(size 1.27 1.27)
+				)
+			)
+		)
+		(property "MPN" "ADBMS6822CCSZ"
+			(at 100.33 115.57 0)
+			(hide yes)
+			(show_name no)
+			(do_not_autoplace no)
+			(effects
+				(font
+					(size 1.27 1.27)
+				)
+			)
+		)
+		(property "MANUFACTURER" "Analog Devices"
+			(at 100.33 115.57 0)
+			(hide yes)

Commit message: Use 1206 on AFEs
Parts:
- removed C37: 10nF, APRL_Passive:C_0603, symbol Device:C_Small
- removed C38, C39, C40: 100nF, APRL_Passive:C_0603, symbol Device:C_Small
- removed J4: Conn_01x06, APRL_Connector_Molex:Molex_CLIK-Mate_503159-0601_1x06-1MP_P1.50mm_Vertical, symbol Connector_Generic:Conn_01x06
- removed R20: 100k, APRL_Passive:R_0603, symbol Device:R_Small_US
- removed U5: ADBMS6822, APRL_Package_QFN:LFCSP-32-1EP_5x5mm_P0.5mm_EP2.1x2.1mm_ThermalVias, symbol APRL_Comms:ADBMS6822
- added J7: Conn_01x04, APRL_Connector_Molex:Molex_CLIK-Mate_503159-0401_1x04-1MP_P1.50mm_Vertical, symbol Connector_Generic:Conn_01x04
- added U5: ADBMS6821, APRL_Package_QFN:LFCSP-32-1EP_5x5mm_P0.5mm_EP2.1x2.1mm_ThermalVias, symbol APRL_Comms:ADBMS6821
- renumbered C36 to C32, C32 to C33, C33 to C34, C34 to C35, C35 to C36
Connections:
- net +3.3V: now also U5.1 (MSTR), U5.14 (PHAPOL), U5.16 (XCVRMD), U5.6 (VDDS)
- net +5V: now also U5.12 (VDD), U5.13 (VP)
- net GND: now also U5.15 (RTO), U5.33 (GND), U5.9 (GND)
- net GNDPWR: now also J7.4 (Pin_4)
- net MISO: now also U5.2 (PICO)
- net SCK: now also U5.4 (SCK)
- net ~{CS}: now also U5.5 (~{CS})
- net at C35.2, C36.1, U6.7 (SEL)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: now also J7.3 (Pin_3)
- net at TR1.16 (TX+): now also J7.2 (Pin_2)
- net at TR1.14 (TX-): now also J7.1 (Pin_1)
- net at R19.1, TR1.1 (TD+): now also U5.11 (IP)
- net at R19.2, TR1.3 (TD-): now also U5.10 (IM)
- new net: U5.17 (NIC), U5.18 (NIC), U5.19 (NIC), U5.20 (NIC), U5.21 (NIC), U5.22 (NIC), U5.23 (NIC), U5.24 (NIC), U5.25 (NIC), U5.26 (NIC), U5.27 (NIC), U5.28 (NIC), U5.29 (NIC), U5.30 (NIC), U5.31 (NIC), U5.32 (NIC)
- new net MOSI: U5.3 (POCI)
- no-connect marks 5 -> 9
Other:
- note added: "SPI Mode 3 for TX, Default timeout for battery operation, 2 Mbps bidirectional with 1 bit shift"
- note removed: "SPI Mode 1 for RX, Default timeout for battery operation, 4 Mbps one-way"
- moved on the sheet: C32, C33, C34, C35, C36, F3, TR1, U6

Commit message: Simplify chickensticks, get isospi-tx ready, and update some cubemx projects
Other:
- moved on the sheet: C29, C30, C31, C32, C33, C34, C35, C36, F3, J7, R19, TR1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
