File: ali/v2/isospi-transceiver/microcontroller.kicad_sch (KiCad schematic)
At the start: 39 parts, among them J1 Conn_02x01, J2 Conn_01x05, J3 USB_C_Receptacle_USB2.0_16P, J6 Screw_Terminal_01x02, SW1 SKRPANE010, U1 STM32H563RIV6, U2 AP2112K-3.3, Y1 25 MHz

Commit message: Big changes (Tim and Daniel review part 1)
Parts:
- J6: footprint Connector_Phoenix_MSTB:PhoenixContact_MSTBV_2,5_2-GF-5,08_1x02_P5.08mm_Vertical_ThreadedFlange_MountHole -> APRL_Connector:PhoenixContact_MSTBV_2,5_2-GF-5,08_1x02_P5.08mm_Vertical_ThreadedFlange_MountHole

Commit message: Some BoM Changes, add fabrication toolkit settings
Parts:
- R1, R2: MPN RC0603FR-075K1L -> AC0603FR-075K1L
- R3, R4, R5, R6, R7: MPN RC0603FR-0710KL -> AC0603FR-0710KL
- U2: MANUFACTURER Didoes Inc. -> Diodes Inc.

Commit message: Use 1206 on AFEs
Parts:
- renumbered J6 to J4

Commit message: Simplify chickensticks, get isospi-tx ready, and update some cubemx projects
Connections:
- net USER_LED_1: now also U1.26 (PB0)
- net USER_LED_2: now also U1.27 (PB1)
- net USER_LED_3: now also U1.35 (PB13)
- net ~{CS}: now reaches U1.56 (PC12)
- net SCK: now reaches U1.57 (PB3(JTDO)
- net MISO: now reaches U1.58 (PB4(NJTRST))
- net MOSI: now reaches U1.59 (PB5)
- no-connect marks 8 -> 35
