File: misc/chickensticks/Power.kicad_sch (KiCad schematic)
At the start: 26 parts, among them J10 Conn_01x03_Pin, Q1 Si2371EDS, Q2 DMG9926UDM, U5 LP5907MFX-3.3, U6 MCP73831-2-MC, U7 BQ29700

Commit message: Simplify chickensticks, get isospi-tx ready, and update some cubemx projects
Parts:
- removed BT1: 18650, Battery:BatteryHolder_Keystone_1042_1x18650, symbol Device:Battery_Cell
- removed C26, C27, C28, C29, C30, C31: 22uF, APRL_Passive:C_0805, symbol Device:C_Small
- removed C32: 100nF, APRL_Passive:C_0603, symbol Device:C_Small
- removed D10, D11, D9: LED_Small, APRL_Passive:LED_0603, symbol Device:LED_Small
- removed F2: 250mA, APRL_Passive:Fuse_0805_2012Metric, symbol Device:Fuse_Small
- removed J10: Conn_01x03_Pin, Connector_PinHeader_2.54mm:PinHeader_1x03_P2.54mm_Vertical, symbol Connector:Conn_01x03_Pin
- removed Q1: Si2371EDS, Package_TO_SOT_SMD:SOT-23, symbol Transistor_FET:Si2371EDS
- removed Q2: DMG9926UDM, Package_TO_SOT_SMD:SOT-23-6, symbol Transistor_FET:DMG9926UDM
- removed R11, R12, R15: 10k, APRL_Passive:R_0603, symbol Device:R_Small_US
- removed R13: 100R, APRL_Passive:R_0603, symbol Device:R_Small_US
- removed R14: 100k, APRL_Passive:R_0603, symbol Device:R_Small_US
- removed R16: 330R, APRL_Passive:R_0603, symbol Device:R_Small_US
- removed R17: 2k, APRL_Passive:R_0603, symbol Device:R_Small_US
- removed R18: 2.2k, APRL_Passive:R_0603, symbol Device:R_Small_US
- removed U5: LP5907MFX-3.3, Package_TO_SOT_SMD:SOT-23-5, symbol Regulator_Linear:LP5907MFX-3.3
- removed U6: MCP73831-2-MC, APRL_Package:DFN-8-1EP_3x2mm_P0.5mm_EP1.7x1.4mm, symbol APRL_Power:MCP73831-2-MC
- removed U7: BQ29700, Package_SON:WSON-6_1.5x1.5mm_P0.5mm, symbol Battery_Management:BQ297xy
Connections:
- no-connect marks 1 -> 0
Other:
- note removed: "+3.3V RF LDO"
- note removed: "+3.3V Selector"
- note removed: "Cell Protection + Charging"
- note removed: "Configured for max charging at 500mA (This will take awhile to charge and get hot)"
- note removed: "Power"
- note removed: "Rail switching mechanism: 1. Prevents backflow from battery to USB 2. Battery connected with USB is not 3. If USB is connected, the battery charger IC only powers the lithium cell"
- note removed: "This is going to drop out for the last ~20% of the battery, then RF performance will likely be degraded"
- company: Aggie Propulsion & Rocketry Lab -> (none)
- title: Chickenstick -> (none)
